File: kicad/single_din_bottom_rev_a.kicad_pcb (KiCad board)
At the start: 2 copper layers, 86 x 14 mm, 7 parts, among them J1 Conn_01x04, J2 Conn_01x04, J3 Conn_01x04, J4 Conn_01x04, U1 R-78B3.3-1.0 (Recom)

Commit message: Added self power possibilities
Parts:
- added R1: 0R, Resistor_SMD:R_0805_2012Metric, B.Cu at (96.1, 169.0)
- added R2: 0R, Resistor_SMD:R_0805_2012Metric, B.Cu at (96.0, 172.9)
Routing:
- net /Vin: track 33.2 -> 59.3 mm
- net /Vout: track 47.2 -> 66.3 mm
- net /IO1: track 21.3 -> 33.5 mm
Changed lines of the file:
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@@
     (thickness 1.6)
     (drawings 10)
-    (tracks 32)
+    (tracks 45)
     (zones 0)
-    (modules 7)
+    (modules 9)
     (nets 10)
   )
@@
     (add_net "Net-(J1-Pad2)")
     (add_net "Net-(J1-Pad3)")
+  )
+  (module Resistor_SMD:R_0805_2012Metric (layer B.Cu)
+    (at 95.9739 172.8597 180)
+    (descr "Resistor SMD 0805 (2012 Metric), square (rectangular) end terminal, IPC_7351 nominal, (Body size source: IPC-SM-782 page 72, https://www.pcb-3d.com/wordpress/wp-content/uploads/ipc-sm-782a_amendment_1_and_2.pdf), generated with kicad-footprint-generator")
+    (tags resistor)
+    (attr smd)
+    (fp_text reference R2 (at 0 1.65) (layer B.SilkS)
+      (effects (font (size 1 1) (thickness 0.15)) (justify mirror))
+    )
+    (fp_text value 0R (at 0 -1.65) (layer B.Fab)
+      (effects (font (size 1 1) (thickness 0.15)) (justify mirror))
+    )
+    (fp_text user %R (at 0 0) (layer B.Fab)
+      (effects (font (size 0.5 0.5) (thickness 0.08)) (justify mirror))
+    )
+    (fp_line (start -1 -0.625) (end -1 0.625) (layer B.Fab) (width 0.1))
+    (fp_line (start -1 0.625) (end 1 0.625) (layer B.Fab) (width 0.1))
+    (fp_line (start 1 0.625) (end 1 -0.625) (layer B.Fab) (width 0.1))
+    (fp_line (start 1 -0.625) (end -1 -0.625) (layer B.Fab) (width 0.1))
+    (fp_line (start -0.227064 0.735) (end 0.227064 0.735) (layer B.SilkS) (width 0.12))
+    (fp_line (start -0.227064 -0.735) (end 0.227064 -0.735) (layer B.SilkS) (width 0.12))
+    (fp_line (start -1.68 -0.95) (end -1.68 0.95) (layer B.CrtYd) (width 0.05))
+    (fp_line (start -1.68 0.95) (end 1.68 0.95) (layer B.CrtYd) (width 0.05))
+    (fp_line (start 1.68 0.95) (end 1.68 -0.95) (layer B.CrtYd) (width 0.05))
+    (fp_line (start 1.68 -0.95) (end -1.68 -0.95) (layer B.CrtYd) (width 0.05))
+    (pad 2 smd roundrect (at 0.9125 0 180) (size 1.025 1.4) (layers B.Cu B.Paste B.Mask) (roundrect_rratio 0.243902)
+      (net 2 /Vin))
+    (pad 1 smd roundrect (at -0.9125 0 180) (size 1.025 1.4) (layers B.Cu B.Paste B.Mask) (roundrect_rratio 0.243902)
+      (net 9 /IO1))
+    (model ${KISYS3DMOD}/Resistor_SMD.3dshapes/R_0805_2012Metric.wrl
+      (at (xyz 0 0 0))
+      (scale (xyz 1 1 1))
+      (rotate (xyz 0 0 0))
+    )
+  )
+  (module Resistor_SMD:R_0805_2012Metric (layer B.Cu)
+    (at 96.0501 168.9989 180)
+    (descr "Resistor SMD 0805 (2012 Metric), square (rectangular) end terminal, IPC_7351 nominal, (Body size source: IPC-SM-782 page 72, https://www.pcb-3d.com/wordpress/wp-content/uploads/ipc-sm-782a_amendment_1_and_2.pdf), generated with kicad-footprint-generator")
+    (tags resistor)
+    (attr smd)
+    (fp_text reference R1 (at 0 1.65) (layer B.SilkS)
+      (effects (font (size 1 1) (thickness 0.15)) (justify mirror))
+    )
+    (fp_text value 0R (at 0 -1.65) (layer B.Fab)
+      (effects (font (size 1 1) (thickness 0.15)) (justify mirror))
+    )
+    (fp_line (start 1.68 -0.95) (end -1.68 -0.95) (layer B.CrtYd) (width 0.05))
+    (fp_line (start 1.68 0.95) (end 1.68 -0.95) (layer B.CrtYd) (width 0.05))
+    (fp_line (start -1.68 0.95) (end 1.68 0.95) (layer B.CrtYd) (width 0.05))
+    (fp_line (start -1.68 -0.95) (end -1.68 0.95) (layer B.CrtYd) (width 0.05))
+    (fp_line (start -0.227064 -0.735) (end 0.227064 -0.735) (layer B.SilkS) (width 0.12))
+    (fp_line (start -0.227064 0.735) (end 0.227064 0.735) (layer B.SilkS) (width 0.12))
+    (fp_line (start 1 -0.625) (end -1 -0.625) (layer B.Fab) (width 0.1))
+    (fp_line (start 1 0.625) (end 1 -0.625) (layer B.Fab) (width 0.1))
+    (fp_line (start -1 0.625) (end 1 0.625) (layer B.Fab) (width 0.1))
+    (fp_line (start -1 -0.625) (end -1 0.625) (layer B.Fab) (width 0.1))
+    (fp_text user %R (at 0 0) (layer B.Fab)
+      (effects (font (size 0.5 0.5) (thickness 0.08)) (justify mirror))
+    )
+    (pad 2 smd roundrect (at 0.9125 0 180) (size 1.025 1.4) (layers B.Cu B.Paste B.Mask) (roundrect_rratio 0.243902)
+      (net 3 /Vout))
+    (pad 1 smd roundrect (at -0.9125 0 180) (size 1.025 1.4) (layers B.Cu B.Paste B.Mask) (roundrect_rratio 0.243902)
+      (net 9 /IO1))
+    (model ${KISYS3DMOD}/Resistor_SMD.3dshapes/R_0805_2012Metric.wrl
+      (at (xyz 0 0 0))
+      (scale (xyz 1 1 1))
+      (rotate (xyz 0 0 0))
+    )
   )
   (module Converter_DCDC:Converter_DCDC_RECOM_R-78B-2.0_THT (layer F.Cu)
@@
   (segment (start 59.7408 168.5417) (end 59.7408 169.8752) (width 1) (layer F.Cu) (net 2))
   (segment (start 60.8711 167.4114) (end 59.7408 168.5417) (width 1) (layer F.Cu) (net 2))
+  (segment (start 72.0598 170.8044) (end 72.0598 168.5544) (width 1) (layer B.Cu) (net 2))
+  (segment (start 74.1151 172.8597) (end 72.0598 170.8044) (width 1) (layer B.Cu) (net 2))
+  (segment (start 95.0614 172.8597) (end 74.1151 172.8597) (width 1) (layer B.Cu) (net 2))
   (segment (start 77.1398 175.895) (end 77.1398 168.5544) (width 1) (layer F.Cu) (net 3))
   (segment (start 50.0761 179.2097) (end 73.8251 179.2097) (width 1) (layer F.Cu) (net 3))
@@
   (segment (start 84.3534 168.5544) (end 86.0044 170.2054) (width 1) (layer F.Cu) (net 3))
   (segment (start 77.1398 168.5544) (end 84.3534 168.5544) (width 1) (layer F.Cu) (net 3))
+  (segment (start 95.1376 168.9989) (end 92.4814 168.9989) (width 1) (layer B.Cu) (net 3))
+  (segment (start 92.4814 168.9989) (end 90.9066 167.4241) (width 1) (layer B.Cu) (net 3))
+  (segment (start 90.9066 167.4241) (end 85.4202 167.4241) (width 1) (layer B.Cu) (net 3))
+  (segment (start 84.2899 168.5544) (end 77.1398 168.5544) (width 1) (layer B.Cu) (net 3))
+  (segment (start 85.4202 167.4241) (end 84.2899 168.5544) (width 1) (layer B.Cu) (net 3))
   (segment (start 41.402 171.7802) (end 51.1556 171.7802) (width 1) (layer F.Cu) (net 4))
   (segment (start 52.1716 172.7962) (end 52.1716 177.4952) (width 1) (layer F.Cu) (net 4))
@@
   (segment (start 92.5576 169.0116) (end 104.7242 169.0116) (width 1) (layer F.Cu) (net 9))
   (segment (start 91.186 170.3832) (end 92.5576 169.0116) (width 1) (layer F.Cu) (net 9))
+  (segment (start 104.7115 168.9989) (end 104.7242 169.0116) (width 1) (layer B.Cu) (net 9))
+  (segment (start 96.8864 170.2327) (end 98.1202 168.9989) (width 1) (layer B.Cu) (net 9))
+  (segment (start 96.8864 172.8597) (end 96.8864 170.2327) (width 1) (layer B.Cu) (net 9))
+  (segment (start 98.1202 168.9989) (end 104.7115 168.9989) (width 1) (layer B.Cu) (net 9))
+  (segment (start 96.9626 168.9989) (end 98.1202 168.9989) (width 1) (layer B.Cu) (net 9))
   (zone (net 1) (net_name GND) (layer F.Cu) (hatch edge 0.508)
     (connect_pads (clearance 0.508))
@@
     (polygon
       (pts
-        (xy 115.7224 166.1541) (xy 116.0145 179.7812) (xy 30.0609 180.0606) (xy 30.2133 166.0144)
+        (xy 115.5954 166.2938) (xy 115.8113 179.705) (xy 30.1117 179.705) (xy 29.9339 166.0144)
       )
     )
