File: kicad/single_din_bottom.kicad_pcb (KiCad board)
At the start: 2 copper layers, 86 x 14 mm, 9 parts, among them J1 Conn_01x04, J2 Conn_01x04, J3 Conn_01x04, J4 Conn_01x04, U1 R-78B3.3-1.0 (Recom)

Commit message: Fixed ground plane
Routing:
- net GND: vias 0 -> 2

Commit message: Fixed som design errors
Other:
- net class Default removed
